File: besspin/cyberPhys/hardware/Physical Architecture Diagram/CYBERPHYS_DEMONSTRATOR_ARCHITECTURE_PHYSICAL_REV_D.sch (EAGLE design)
At the start: 47 parts

Commit message: Added LED Manager Board and Physical System Architecture Updates
Parts:
- removed DEBOUNCER1: (no value), USER_GALOIS_CYBERPHYS:RELAY_CONTACT_DEBOUNCER
- removed FADECANDY1: ADAFRUIT 1689 (ASIN B00K9M3VLE), USER_GALOIS_CYBERPHYS:FADECANDY_LED_DRIVER
- removed LED_STRING1, LED_STRING2, LED_STRING3, LED_STRING4, LED_STRING5, LED_STRING6, LED_STRING7, LED_STRING8: WS2815, USER_GALOIS_CYBERPHYS:WS2815_LED_STRING
- removed POWER_SUPPLY1: MEANWELL HRP-450-12, USER_GALOIS_CYBERPHYS:POWER_SUPPLY_BULK
- removed RELAY1: SMAKN LCUS-1 (ASIN B01CN7E0RQ), USER_GALOIS_CYBERPHYS:USB_RELAY
- removed TERMINAL_BLOCK1: (no value), USER_GALOIS_CYBERPHYS:TERMINAL_BLOCK
- removed USB_HUB3: (no value), USER_GALOIS_CYBERPHYS:USB_HUB_1X10
- added FADECANDY2: ADAFRUIT 1689 (ASIN B00K9M3VLE), USER_GALOIS_CYBERPHYS:FADECANDY_LED_DRIVER
- added LED_STRING10, LED_STRING11, LED_STRING12, LED_STRING13, LED_STRING14, LED_STRING15, LED_STRING16, LED_STRING9: WS2815, USER_GALOIS_CYBERPHYS:WS2815_LED_STRING
- added PCBA1: (no value), USER_GALOIS_CYBERPHYS:PCBA_LED_MANAGER
- added RELAY2, RELAY3: SMAKN LCUS-1 (ASIN B01CN7E0RQ), USER_GALOIS_CYBERPHYS:USB_RELAY
- added U$32: FANATEC_PODIUM_KILL_SWITCH, USER_GALOIS_CYBERPHYS:FANATEC_PODIUM_KILL_SWITCH
- added U$33: SMARTCAR_THERMOMETER, USER_GALOIS_CYBERPHYS:SMARTCAR_THERMOMETER
- added USB_HUB4: (no value), USER_GALOIS_CYBERPHYS:USB_HUB_1X10
- PC1: PROCESS1 BeamNG.research -> BeamNG.tech; PROCESS2 ignition.py -> Ignition ecosystem
Connections:
- removed net +12V_SWITCHED: DEBOUNCER1.VIN, RELAY1.VOUT
- removed net +12V_SWITCHED_DEBOUNCED: DEBOUNCER1.VOUT, TERMINAL_BLOCK1.VIN
- removed net FADECANDY_CTRL_0: FADECANDY1.0, LED_STRING1.CTRL
- removed net FADECANDY_CTRL_1: FADECANDY1.1, LED_STRING2.CTRL
- removed net FADECANDY_CTRL_2: FADECANDY1.2, LED_STRING3.CTRL
- removed net FADECANDY_CTRL_3: FADECANDY1.3, LED_STRING4.CTRL
- removed net FADECANDY_CTRL_4: FADECANDY1.4, LED_STRING5.CTRL
- removed net FADECANDY_CTRL_5: FADECANDY1.5, LED_STRING6.CTRL
- removed net FADECANDY_CTRL_6: FADECANDY1.6, LED_STRING7.CTRL
- removed net FADECANDY_CTRL_7: FADECANDY1.7, LED_STRING8.CTRL
- removed net N$10: LED_STRING2.+12V, TERMINAL_BLOCK1.VOUT@2
- removed net N$11: LED_STRING3.+12V, TERMINAL_BLOCK1.VOUT@3
- removed net N$12: LED_STRING4.+12V, TERMINAL_BLOCK1.VOUT@4
- removed net N$13: LED_STRING5.+12V, TERMINAL_BLOCK1.VOUT@5
- removed net N$14: LED_STRING6.+12V, TERMINAL_BLOCK1.VOUT@6
- removed net N$15: LED_STRING7.+12V, TERMINAL_BLOCK1.VOUT@7
- removed net N$16: LED_STRING8.+12V, TERMINAL_BLOCK1.VOUT@8
- removed net N$9: LED_STRING1.+12V, TERMINAL_BLOCK1.VOUT@1
- removed net USB_FADECANDY: FADECANDY1.USB, USB_HUB3.USB2
- removed net USB_RELAY_LED_+12V: RELAY1.USB, USB_HUB3.USB1
- new net AC/DC_KANTO_YU2: SPEAKERS1.VDC
- new net KILL_SWITCH_RJ12_CABLE: U$32.P$1, WHEEL_BASE1.E-STOP
- new net N$17: CLUSTER1.TEMP, U$33.P$1
- new net N$18: LED_STRING9.+12V, LED_STRING9.CTRL, PCBA1.LED0
- new net N$19: LED_STRING10.+12V, LED_STRING10.CTRL, PCBA1.LED1
- new net N$20: LED_STRING11.+12V, LED_STRING11.CTRL, PCBA1.LED2
- new net N$21: LED_STRING12.+12V, LED_STRING12.CTRL, PCBA1.LED3
- new net N$22: RELAY3.VOUT, U$44.PWR_+12V
- new net N$23: LED_STRING13.+12V, LED_STRING13.CTRL, PCBA1.LED4
- new net N$24: LED_STRING14.+12V, LED_STRING14.CTRL, PCBA1.LED5
- new net N$25: LED_STRING15.+12V, LED_STRING15.CTRL, PCBA1.LED6
- new net N$27: LED_STRING16.+12V, LED_STRING16.CTRL, PCBA1.LED7
- new net USB_FADECANDY2: FADECANDY2.USB, USB_HUB4.USB2
- new net USB_RELAY2_LED_+12V: RELAY2.USB, USB_HUB4.USB1
- new net USB_TEENSY_PWR_CTRL: PC2.USB2, RELAY3.USB
- net +12V_BULK: now also PCBA1.+12VDC, RELAY3.VIN; no longer POWER_SUPPLY1.DC_OUT, RELAY1.VIN, U$44.PWR_+12V
- net 110VAC: no longer POWER_SUPPLY1.AC_IN, SPEAKERS1.VAC
- net USB_LED_NETWORK_CTRL: now also USB_HUB4.USB_EXT; no longer USB_HUB3.USB_EXT
- net USB_LED_NETWORK_DC: now also USB_HUB4.PWR; no longer USB_HUB3.PWR
Other:
- note added: "EXAMPLE LED STRING BANK CONTROL AND POWER SETUP WITH LED MANAGER PCBA"
- note added: "RJ12 CABLE"
- note removed: "EXAMPLE LED STRING BANK CONTROL AND POWER SETUP"
- note removed: "RJ45 CABLE"
